File: hardware/fanctl.kicad_sch (KiCad schematic)
At the start: 10 parts, among them J501 4PIN FANCTL, Q501 2N7002K, Q502 SSM3J332R

Commit message: Changed OpAMP part no.
Parts:
- J501: digikey (none) -> WM4330-ND; distributor (none) -> https://www.digikey.jp/en/products/detail/molex/0470531000/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
Changed lines of the file:
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@@
+			)
+		)
+		(property "digikey" "WM4330-ND"
+			(at 219.71 95.25 0)
+			(effects
+				(font
+					(size 1.27 1.27)
+				)
+				(hide yes)
+			)
+		)
+		(property "distributor" "https://www.digikey.jp/en/products/detail/molex/0470531000/2421261"
+			(at 219.71 95.25 0)
+			(effects
+				(font
+					(size 1.27 1.27)
+				)
+				(hide yes)
 			)
 		)
